File: hw/start.sch (EAGLE design)
At the start: 3 parts, among them U1 ESP32-DEVKITC-32D

Commit message: x
Parts:
- added S1: MOMENTARY-SWITCH-SPST-PTH-6.0MM, SparkFun-Switches:MOMENTARY-SWITCH-SPST-PTH-6.0MM
Connections:
- new net N$4: S1.1, U1.SD3
- net N$3: now also S1.2
Changed lines of the file:
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@@
 <part name="R1" library="resistor" library_urn="urn:adsk.eagle:library:348" deviceset="R-EU_" device="0204/5" package3d_urn="urn:adsk.eagle:package:23488/1" value="2k"/>
 <part name="D1" library="SparkFun-LED" library_urn="urn:adsk.eagle:library:529" deviceset="LED" device="5MM" package3d_urn="urn:adsk.eagle:package:39353/1"/>
+<part name="S1" library="SparkFun-Switches" library_urn="urn:adsk.eagle:library:535" deviceset="MOMENTARY-SWITCH-SPST" device="-PTH-6.0MM" package3d_urn="urn:adsk.eagle:package:40163/1" value=""/>
 </parts>
 <sheets>
@@
 <attribute name="NAME" x="85.852" y="65.151" size="1.778" layer="95" font="vector" rot="R180"/>
 <attribute name="VALUE" x="85.852" y="70.485" size="1.778" layer="96" font="vector" rot="R180" align="top-left"/>
+</instance>
+<instance part="S1" gate="G$1" x="71.12" y="35.56" smashed="yes">
+<attribute name="NAME" x="71.12" y="37.084" size="1.778" layer="95" font="vector" align="bottom-center"/>
+<attribute name="VALUE" x="71.12" y="35.052" size="1.778" layer="96" font="vector" align="top-center"/>
 </instance>
 </instances>
@@
 <pinref part="D1" gate="G$1" pin="C"/>
 <wire x1="88.9" y1="68.58" x2="86.36" y2="68.58" width="0.1524" layer="91"/>
+<wire x1="88.9" y1="68.58" x2="88.9" y2="35.56" width="0.1524" layer="91"/>
+<junction x="88.9" y="68.58"/>
+<pinref part="S1" gate="G$1" pin="2"/>
+<wire x1="76.2" y1="35.56" x2="88.9" y2="35.56" width="0.1524" layer="91"/>
 </segment>
 </net>
+<net name="N$4" class="0">
+<segment>
+<pinref part="U1" gate="G$1" pin="SD3"/>
+<wire x1="22.86" y1="50.8" x2="17.78" y2="50.8" width="0.1524" layer="91"/>
+<wire x1="17.78" y1="50.8" x2="17.78" y2="35.56" width="0.1524" layer="91"/>
+<pinref part="S1" gate="G$1" pin="1"/>
+<wire x1="66.04" y1="35.56" x2="17.78" y2="35.56" width="0.1524" layer="91"/>
+</segment>
+</net>
